File: pcb/uvProject_v2/uvProject_v2.kicad_pcb (KiCad board)
At the start: 2 copper layers, 70 x 70 mm, 22 parts, among them J1 RTC Module, J2 RESET, J3 UART, J4 BOOT, J5 POWER, J6 UV sensor, J7 Micro SD, U1 LM1117-3.3, U2 ESP8266-12E/ESP-12E

Commit message: update:pcb
Parts:
- added R7: 10K, Resistor_SMD:R_1206_3216Metric_Pad1.30x1.75mm_HandSolder, B.Cu at (172.2, 104.7)
- added R8: 10K, Resistor_SMD:R_1206_3216Metric_Pad1.30x1.75mm_HandSolder, B.Cu at (174.7, 104.7)
- added R9: 10K, Resistor_SMD:R_1206_3216Metric_Pad1.30x1.75mm_HandSolder, B.Cu at (160.4, 111.8)
- C3: moved to F.Cu
- C4: value 10u -> 100u
- R10: renamed from R7; value 22K -> 10K
- moved R10 17.7 mm to (154.7, 111.8), turned to 180 degrees
- moved R2 4.00 mm to (169.7, 104.7)
- moved R3 0.60 mm to (177.2, 104.7)
- moved R1 0.30 mm to (179.6, 104.7)
Connections:
- R10 pad 1: /DATA -> Net-(R10-Pad1)
Routing:
- net /DeepSleep: track 110.9 -> 15.8 mm
- net +3.3V: track 236.5 -> 256.9 mm
- net Net-(J6-Pin_2): track 23.2 -> 3.12 mm
- net Net-(R7-Pad2): track 0.00 -> 15.1 mm
- net /DATA: track 15.7 -> 3.63 mm, vias 2 -> 0
- net GND: track 31.8 -> 24.4 mm, vias 16 -> 12
- net Net-(R10-Pad1): track 0.00 -> 2.60 mm
- net Net-(U2-EN): track 8.50 -> 10.2 mm
- added copper zone on B.Cu, net /DATA
Other:
- board text added: "v1.02"
